Commit message: new

File: src/nashbot/description/robot.urdf (robot description, URDF)
Before this commit: robot nashbot, 29 links, 28 joints
Links:
- removed link caster
- removed link caster_2
- added link t_2-2_mouting_plate, mass 0.038153138865978875049; collision mesh filename=package://nashbot/description/t_2-2_mouting_plate.stl; visual mesh filename=package://nashbot/description/t_2-2_mouting_plate.stl
- added link t_2-2_mouting_plate_2, mass 0.038153138865978875049; collision mesh filename=package://nashbot/description/t_2-2_mouting_plate.stl; visual mesh filename=package://nashbot/description/t_2-2_mouting_plate.stl
- added link t_2-3_bracket, mass 0.030960253599026488214; collision mesh filename=package://nashbot/description/t_2-3_bracket.stl; visual mesh filename=package://nashbot/description/t_2-3_bracket.stl
- added link t_2-3_bracket_2, mass 0.030960253599026488214; collision mesh filename=package://nashbot/description/t_2-3_bracket.stl; visual mesh filename=package://nashbot/description/t_2-3_bracket.stl
- added link t_2-3_bracket_3, mass 0.030960253599026488214; collision mesh filename=package://nashbot/description/t_2-3_bracket.stl; visual mesh filename=package://nashbot/description/t_2-3_bracket.stl
- added link t_2-3_bracket_4, mass 0.030960253599026488214; collision mesh filename=package://nashbot/description/t_2-3_bracket.stl; visual mesh filename=package://nashbot/description/t_2-3_bracket.stl
- added link t_2-4_wheel, mass 0.18421750729180022543; collision mesh filename=package://nashbot/description/t_2-4_wheel.stl; visual mesh filename=package://nashbot/description/t_2-4_wheel.stl
- added link t_2-4_wheel_2, mass 0.18421750729180022543; collision mesh filename=package://nashbot/description/t_2-4_wheel.stl; visual mesh filename=package://nashbot/description/t_2-4_wheel.stl
- added link t_2-5_tire, mass 0.01273663756489323666; collision mesh filename=package://nashbot/description/t_2-5_tire.stl; visual mesh filename=package://nashbot/description/t_2-5_tire.stl
- added link t_2-5_tire_2, mass 0.01273663756489323666; collision mesh filename=package://nashbot/description/t_2-5_tire.stl; visual mesh filename=package://nashbot/description/t_2-5_tire.stl
- added link t_2-6_pin, mass 0.015325915748070038924; collision mesh filename=package://nashbot/description/t_2-6_pin.stl; visual mesh filename=package://nashbot/description/t_2-6_pin.stl
- added link t_2-6_pin_2, mass 0.015325915748070038924; collision mesh filename=package://nashbot/description/t_2-6_pin.stl; visual mesh filename=package://nashbot/description/t_2-6_pin.stl
- link link_arm1_bearing: mass 0.060475658581603586317 -> 0.060475658581603579378
- link link_arm3: mass 0.12431354679013274789 -> 0.12431354679013277564
- link link_arm4: mass 0.12168204910675756159 -> 0.12168204910675753383
- link link_arm_wrist2: mass 0.0076395059073011539058 -> 0.0076395059073011530384
- link link_base: mass 6.9241979448356403282 -> 6.92419794483562967
- link link_wrist_base: mass 0.01299711733361526636 -> 0.012997117333615264625
- link link_wrist_base_bearing: mass 0.0023389497908041689996 -> 0.0023389497908041681322
- link link_wrist_end: mass 0.017319283609535648938 -> 0.017319283609535641999
- link link_wrist_mid: mass 0.025315413537536853722 -> 0.025315413537536850253
Joints:
- added joint caster_axle: type continuous, parent t_2-3_bracket, child t_2-6_pin, origin xyz=-0.019641819999999997337 0 -0.036182300000000000573 rpy=1.570796326794896558 -1.3877677137361563236e-14 -3.1225022567581769653e-17, axis 0 0 1, limit effort=1 velocity=20
- added joint caster_axle2: type continuous, parent t_2-3_bracket_3, child t_2-6_pin_2, origin xyz=-0.019641820000000004276 -1.3877787807814456755e-17 -0.036182300000000000573 rpy=1.570796326794896558 1.0769274009316926161e-14 8.2714011591809387361e-29, axis 0 0 1, limit effort=1 velocity=20
- added joint caster_inner_axle: type continuous, parent t_2-6_pin, child t_2-4_wheel, origin xyz=1.3877787807814456755e-17 -8.6736173798840354721e-19 -0.011630024999999988289 rpy=3.141592653589793116 2.7755575615629246311e-17 1.570796326794896558, axis 0 0 1, limit effort=1 velocity=20
- added joint caster_inner_axle2: type continuous, parent t_2-6_pin_2, child t_2-4_wheel_2, origin xyz=-2.7755575615628913511e-17 0 -0.011630025000000002167 rpy=3.1415926535897926719 5.3790483572030952479e-16 -2.2447468074446286224, axis 0 0 1, limit effort=1 velocity=20
- added joint caster_shaft: type fixed, parent t_2-2_mouting_plate, child t_2-3_bracket, origin xyz=-0.020675599999999988432 -0.010337800000000008094 -0.0025844499999999742679 rpy=-5.5511151231262005519e-17 -1.1067045303393603349e-19 -3.4694469519546380132e-18, axis 0 0 1, limit effort=1 velocity=20
- added joint caster_shaft2: type fixed, parent t_2-2_mouting_plate, child t_2-3_bracket_2, origin xyz=-0.020675599999999988432 0.010337800000000035849 -0.0025844499999999742679 rpy=-5.5511151231262005519e-17 -1.1067045303393603349e-19 -3.4694469519546380132e-18, axis 0 0 1, limit effort=1 velocity=20
- added joint caster_shaft3: type fixed, parent t_2-2_mouting_plate_2, child t_2-3_bracket_3, origin xyz=-0.020675599999999932921 -0.010337799999999983808 -0.0025844500000000228401 rpy=0 2.7644905162743880414e-17 -2.7755575615620445582e-17, axis 0 0 1, limit effort=1 velocity=20
- added joint caster_shaft4: type fixed, parent t_2-2_mouting_plate_2, child t_2-3_bracket_4, origin xyz=-0.020675599999999988432 0.010337800000000015033 -0.0025844500000000159012 rpy=0 2.7644905162743880414e-17 -2.7755575615620445582e-17, axis 0 0 1, limit effort=1 velocity=20
- added joint caster_wheel: type fixed, parent t_2-4_wheel, child t_2-5_tire, origin xyz=0 0 0 rpy=-3.141592653589793116 -0 0, axis 0 0 1, limit effort=1 velocity=20
- added joint caster_wheel2: type fixed, parent t_2-4_wheel_2, child t_2-5_tire_2, origin xyz=-1.3877787807814456755e-17 -2.7755575615628913511e-17 0 rpy=-3.141592653589793116 1.5808348259625381109e-17 0, axis 0 0 1, limit effort=1 velocity=20
- joint caster_base_mount: child caster -> t_2-2_mouting_plate; origin xyz=-7.5460471204991108607e-17 0.43091411888599395752 -0.039999999999999931444 rpy=7.359732672286190388e-17 1.1896430072343872108e-14 0.0054475775093515916084 -> xyz=-8.6736173798840354721e-18 0.43091411888599395752 -0.039999999999999986955 rpy=5.5511151231256791641e-17 1.4058199049316279774e-14 1.7694179454963328825e-16; type revolute -> continuous
- joint caster_base_mount2: child caster_2 -> t_2-2_mouting_plate_2; origin xyz=-3.4694469519536141888e-18 0 -0.040000000000000007772 rpy=6.4035790008945382877e-15 -2.119918668448466828e-16 1.6038573593312053234 -> xyz=-1.2143064331837649661e-17 0 -0.04000000000000001471 rpy=-6.9365135332916969927e-15 1.1217224233694430174e-15 -1.4123025265630571035; type revolute -> continuous
- joint wheel1_right: type revolute -> continuous
- joint wheel2_left: type revolute -> continuous
