Commit message: new

File: src/nashbot/description/robot.urdf (robot description, URDF)
Before this commit: robot nashbot, 39 links, 38 joints
Links:
- removed link link_camera_servo1
- removed link link_camera_servo2
- removed link link_lead_screw
- removed link link_lead_screw_2
- removed link link_lidar_base_mount
- removed link link_lidar_pole_mount
- removed link link_wheels
- removed link link_wheels_2
- removed link t_2-2_mouting_plate
- removed link t_2-2_mouting_plate_2
- removed link t_2-3_bracket
- removed link t_2-3_bracket_2
- removed link t_2-3_bracket_3
- removed link t_2-3_bracket_4
- removed link t_2-4_wheel
- removed link t_2-4_wheel_2
- removed link t_2-5_tire
- removed link t_2-5_tire_2
- removed link t_2-6_pin
- removed link t_2-6_pin_2
- added link link_cam_v2.1_v1, mass 0.00099893693584445376193; collision mesh filename=package://nashbot/description/link_cam_v2.1_v1.stl; visual mesh filename=package://nashbot/description/link_cam_v2.1_v1.stl
- added link link_cam_v2.1_v1_2, mass 0.00099893693584445376193; collision mesh filename=package://nashbot/description/link_cam_v2.1_v1.stl; visual mesh filename=package://nashbot/description/link_cam_v2.1_v1.stl
- added link link_camera_mount, mass 0.05185638046932426054; collision mesh filename=package://nashbot/description/link_camera_mount.stl; visual mesh filename=package://nashbot/description/link_camera_mount.stl
- added link link_camservo_m1, mass 0.0035384613163860329475; collision mesh filename=package://nashbot/description/link_camservo_m1.stl; visual mesh filename=package://nashbot/description/link_camservo_m1.stl
- added link link_camservo_m2, mass 0.0019317229854466744319; collision mesh filename=package://nashbot/description/link_camservo_m2.stl; visual mesh filename=package://nashbot/description/link_camservo_m2.stl
- added link link_display, mass 0.07400407337253489537; collision mesh filename=package://nashbot/description/link_display.stl; visual mesh filename=package://nashbot/description/link_display.stl
- added link link_esp, mass 0.0028528946071831604372; collision mesh filename=package://nashbot/description/link_esp.stl; visual mesh filename=package://nashbot/description/link_esp.stl
- added link link_extension, mass 0.14831852342676307699; collision mesh filename=package://nashbot/description/link_extension.stl; visual mesh filename=package://nashbot/description/link_extension.stl
- added link link_generic_mount, mass 0.003461874762680981505; collision mesh filename=package://nashbot/description/link_generic_mount.stl; visual mesh filename=package://nashbot/description/link_generic_mount.stl
- added link link_gripper, mass 0.0098904205224396510299; collision mesh filename=package://nashbot/description/link_gripper.stl; visual mesh filename=package://nashbot/description/link_gripper.stl
- added link link_gripper_2, mass 0.0098904205224396510299; collision mesh filename=package://nashbot/description/link_gripper.stl; visual mesh filename=package://nashbot/description/link_gripper.stl
- added link link_gripper_base, mass 0.036747347475539239581; collision mesh filename=package://nashbot/description/link_gripper_base.stl; visual mesh filename=package://nashbot/description/link_gripper_base.stl
- added link link_jetson, mass 0.37117571580316055524; collision mesh filename=package://nashbot/description/link_jetson.stl; visual mesh filename=package://nashbot/description/link_jetson.stl
- added link link_motor_horn, mass 0.0015482237069527797838; collision mesh filename=package://nashbot/description/link_motor_horn.stl; visual mesh filename=package://nashbot/description/link_motor_horn.stl
- added link link_pdb, mass 0.043332218515688546157; collision mesh filename=package://nashbot/description/link_pdb.stl; visual mesh filename=package://nashbot/description/link_pdb.stl
- added link link_planetary_gear_motor, mass 0.16371460908246579513; collision mesh filename=package://nashbot/description/link_planetary_gear_motor.stl; visual mesh filename=package://nashbot/description/link_planetary_gear_motor.stl
- added link link_planetary_gear_motor_2, mass 0.16371460908246579513; collision mesh filename=package://nashbot/description/link_planetary_gear_motor.stl; visual mesh filename=package://nashbot/description/link_planetary_gear_motor.stl
- added link link_planetary_gear_motor_3, mass 0.16371460908246579513; collision mesh filename=package://nashbot/description/link_planetary_gear_motor.stl; visual mesh filename=package://nashbot/description/link_planetary_gear_motor.stl
- added link link_planetary_gear_motor_4, mass 0.16371460908246579513; collision mesh filename=package://nashbot/description/link_planetary_gear_motor.stl; visual mesh filename=package://nashbot/description/link_planetary_gear_motor.stl
- added link link_planetary_gear_motor_5, mass 0.16371460908246579513; collision mesh filename=package://nashbot/description/link_planetary_gear_motor.stl; visual mesh filename=package://nashbot/description/link_planetary_gear_motor.stl
- added link link_planetary_gear_motor_6, mass 0.16371460908246579513; collision mesh filename=package://nashbot/description/link_planetary_gear_motor.stl; visual mesh filename=package://nashbot/description/link_planetary_gear_motor.stl
- added link link_planetary_gear_motor_7, mass 0.16371460908246579513; collision mesh filename=package://nashbot/description/link_planetary_gear_motor.stl; visual mesh filename=package://nashbot/description/link_planetary_gear_motor.stl
- added link link_power_line_mount, mass 0.065027166992509127796; collision mesh filename=package://nashbot/description/link_power_line_mount.stl; visual mesh filename=package://nashbot/description/link_power_line_mount.stl
- added link link_servo_mg, mass 0.26063138106081079615; collision mesh filename=package://nashbot/description/link_servo_mg.stl; visual mesh filename=package://nashbot/description/link_servo_mg.stl
- added link link_servo_mg_2, mass 0.26063138106081079615; collision mesh filename=package://nashbot/description/link_servo_mg.stl; visual mesh filename=package://nashbot/description/link_servo_mg.stl
- added link link_servo_mg_3, mass 0.26063138106081079615; collision mesh filename=package://nashbot/description/link_servo_mg.stl; visual mesh filename=package://nashbot/description/link_servo_mg.stl
- added link link_servo_mg_4, mass 0.26063138106081079615; collision mesh filename=package://nashbot/description/link_servo_mg.stl; visual mesh filename=package://nashbot/description/link_servo_mg.stl
- added link link_ultrasonic, mass 0.00560754301464696462; collision mesh filename=package://nashbot/description/link_ultrasonic.stl; visual mesh filename=package://nashbot/description/link_ultrasonic.stl
- added link link_ultrasonic_2, mass 0.00560754301464696462; collision mesh filename=package://nashbot/description/link_ultrasonic.stl; visual mesh filename=package://nashbot/description/link_ultrasonic.stl
- added link link_ultrasonic_3, mass 0.00560754301464696462; collision mesh filename=package://nashbot/description/link_ultrasonic.stl; visual mesh filename=package://nashbot/description/link_ultrasonic.stl
- added link link_ultrasonic_4, mass 0.00560754301464696462; collision mesh filename=package://nashbot/description/link_ultrasonic.stl; visual mesh filename=package://nashbot/description/link_ultrasonic.stl
- added link link_wheel, mass 0.21292341699643807518; collision mesh filename=package://nashbot/description/link_wheel.stl; visual mesh filename=package://nashbot/description/link_wheel.stl
- added link link_wheel_2, mass 0.21292341699643807518; collision mesh filename=package://nashbot/description/link_wheel.stl; visual mesh filename=package://nashbot/description/link_wheel.stl
- added link link_wheel_3, mass 0.21292341699643807518; collision mesh filename=package://nashbot/description/link_wheel.stl; visual mesh filename=package://nashbot/description/link_wheel.stl
- added link link_wheel_4, mass 0.21292341699643807518; collision mesh filename=package://nashbot/description/link_wheel.stl; visual mesh filename=package://nashbot/description/link_wheel.stl
- added link link_wormgearmotor, mass 0.2858675528412418787; collision mesh filename=package://nashbot/description/link_wormgearmotor.stl; visual mesh filename=package://nashbot/description/link_wormgearmotor.stl
- added link link_wormgearmotor_2, mass 0.2858675528412418787; collision mesh filename=package://nashbot/description/link_wormgearmotor.stl; visual mesh filename=package://nashbot/description/link_wormgearmotor.stl
- added link link_wormgearmotor_3, mass 0.2858675528412418787; collision mesh filename=package://nashbot/description/link_wormgearmotor.stl; visual mesh filename=package://nashbot/description/link_wormgearmotor.stl
- link link_arm1: mass 0.065384397102838151539 -> 0.039230638261702789615
- link link_arm1_base: mass 0.039230638261702789615 -> 0.060390944748639381612
- link link_arm1_bearing: mass 0.060475658581603579378 -> 0.036285395148962132361
- link link_arm1_top_mount: mass 0.24404755337625547162 -> 0.079143117156963080361
- link link_arm2: mass 0.2521046695326249476 -> 0.22334489095979861983
- link link_arm3: mass 0.12431354679013277564 -> 0.11985667013718158402
- link link_arm4: mass 0.12168204910675753383 -> 0.084730816987227688952
- link link_arm_mount_base: mass 0.3476241705557227557 -> 0.34676843776409471687
- link link_arm_wrist2: mass 0.0076395059073011530384 -> 0.015568413400768565599
- link link_armlast: mass 0.023029890215175794627 -> 0.023029890215175791157
- link link_armlast2: mass 0.023029890215175794627 -> 0.029673683675562941703
- link link_base: mass 6.92419794483562967 -> 1.7554185880507504613
- link link_camera: mass 0.38900054186990395966 -> 0.38286436898885872759
- link link_lidar: mass 0.31808625617596653079 -> 0.046857323820461600772
- link link_wrist_base: mass 0.012997117333615264625 -> 0.025071164350844329233
- link link_wrist_end: mass 0.017319283609535641999 -> 0.025188988321725475084
- link link_wrist_mid: mass 0.025315413537536850253 -> 0.025315413537536853722
Joints:
- removed joint arm_base1
- removed joint arm_base_fixed
- removed joint arm_base_mount
- removed joint arm_bearing_mount
- removed joint arm_link2_mount
- removed joint arm_link2_mount2
- removed joint arm_wrist1
- removed joint arm_wrist2
- removed joint arm_wrist2_mount
- removed joint arm_wrist3
- removed joint arm_wrist_fix_mount
- removed joint camera_mount
- removed joint camera_mount1
- removed joint camera_mount2
- removed joint camera_pole
- removed joint caster_axle
- removed joint caster_axle2
- removed joint caster_base_mount
- removed joint caster_base_mount2
- removed joint caster_inner_axle
- removed joint caster_inner_axle2
- removed joint caster_shaft
- removed joint caster_shaft2
- removed joint caster_shaft3
- removed joint caster_shaft4
- removed joint caster_wheel
- removed joint caster_wheel2
- removed joint lidar_base
- removed joint lidar_mount
- removed joint lidar_plate
- removed joint link1.5
- removed joint link2
- removed joint slider_bearing
- removed joint slider_bearing2
- removed joint wheel1_right
- removed joint wheel2_left
- added joint arm_base_top_mount: type fixed, parent link_arm1_top_mount, child link_arm2, origin xyz=1.3877787807814456755e-17 5.2041704279304212832e-18 -0.0049999999999999905631 rpy=-4.7523348266081185674e-17 -4.7545853266420812192e-17 3.1415926535897926719, axis 0 0 1, limit effort=1 velocity=20
- added joint arm_camera: type fixed, parent link_armlast2, child link_cam_v2.1_v1, origin xyz=2.7755575615628913511e-17 0.041864549620449442724 -0.019999999999999684697 rpy=-2.1677104555805458855e-14 -1.1102230246251333676e-16 -1.57079632679489678, axis 0 0 1, limit effort=1 velocity=20
- added joint arm_lowermost_bearing: type fixed, parent link_arm1_base, child link_arm1, origin xyz=-6.9388939039072283776e-18 0.067724570631980882118 -0.012500000000000170697 rpy=1.0560604332947878811e-16 -0 -5.5511151231244989543e-17, axis 0 0 1, limit effort=1 velocity=20
- added joint armplate_baseplate: type fixed, parent link_base, child link_arm_mount_base, origin xyz=-0.033679080195723867797 -0.10384444065391673639 0.0099999999999997851025 rpy=3.141592653589793116 -4.2598488881935332536e-29 -2.6303198217458827823e-28, axis 0 0 1, limit effort=1 velocity=20
- added joint back_left_motor_mount: type fixed, parent link_base, child link_planetary_gear_motor_3, origin xyz=0.20110581606625849149 0.17115555934607412647 -0.010000000000000230926 rpy=1.570796326794896558 -9.4663308626523462545e-30 1.5707963267948972241, axis 0 0 1, limit effort=1 velocity=20
- added joint back_left_wheel: type continuous, parent link_planetary_gear_motor_3, child link_wheel_3, origin xyz=2.7755575615628913511e-17 0.00013236607255451282583 0.024199999999999971534 rpy=-3.1415926535897300553 7.9062755715504319236e-16 -0.013799414977259887027, axis 0 0 1, limit effort=1 velocity=20
- added joint back_right_motor_mount: type fixed, parent link_base, child link_planetary_gear_motor_2, origin xyz=-0.27889418393372578109 0.17115555934607420974 -0.010000000000000008882 rpy=-1.570796326794896558 -6.3108872417683060394e-30 1.570796326794896558, axis 0 0 1, limit effort=1 velocity=20
- added joint back_right_wheel: type continuous, parent link_planetary_gear_motor_2, child link_wheel_2, origin xyz=-0.0067500000000000059952 -2.2204460492503130808e-16 0.024199999999999999289 rpy=3.0878871338032691087e-15 2.0073922473881030536e-14 1.8062615792804408432, axis 0 0 1, limit effort=1 velocity=20
- added joint base_bearing: type revolute, parent link_arm1, child link_arm1_bearing, origin xyz=-7.6327832942979512154e-17 -0.067724570631980798852 -0.015000000000000020262 rpy=-4.1079776914178391981e-22 -3.6499615568547588071e-17 1.8540534590536739135, axis 0 0 1, limit lower=-2.0943951023931952626 upper=2.0943951023931952626 effort=1 velocity=20
- added joint camera_front: type fixed, parent link_generic_mount, child link_cam_v2.1_v1_2, origin xyz=-2.7755575615628913511e-17 -0.015125345474481577401 -0.015851898188250456573 rpy=-1.57079632679489678 1.570796326794896558 0, axis 0 0 1, limit effort=1 velocity=20
- added joint camera_front_mount: type fixed, parent link_arm_mount_base, child link_generic_mount, origin xyz=-3.4256714071673188826e-06 0.086666588097217348019 -0.01000000000000027256 rpy=-1.3550772563145184417e-16 -2.8746819834257579446e-17 -3.141592653589793116, axis 0 0 1, limit effort=1 velocity=20
- added joint depthcam: type fixed, parent link_camservo_m2, child link_camera, origin xyz=-1.6345413365592698085e-06 -0.029231937913894612269 -0.013222478037231732637 rpy=-1.5707963267948996666 1.570796326794896558 0, axis 0 0 1, limit effort=1 velocity=20
- added joint depthcam_link1: type revolute, parent link_servo_mg, child link_camservo_m1, origin xyz=-6.9388939039072283776e-18 -0.010150000000000006239 -0.044750000000000123013 rpy=-2.9184472069012738334e-16 2.6922340728521836213e-16 0.97275063961304364391, axis 0 0 1, limit lower=-1.570796326794896558 upper=1.570796326794896558 effort=1 velocity=20
- added joint depthcam_link2: type revolute, parent link_servo_mg_2, child link_camservo_m2, origin xyz=1.3877787807814456755e-17 1.1102230246251565404e-16 0.0035500000000000140818 rpy=-3.141592653589788231 -3.9881607083193811201e-15 1.8819956131529709253, axis 0 0 1, limit lower=-1.570796326794896558 upper=1.570796326794896558 effort=1 velocity=20
- added joint depthcam_mount: type fixed, parent link_base, child link_camera_pole, origin xyz=-0.035165634782156757199 0.074728912423014520749 0.010000000000000008882 rpy=3.141592653589793116 -4.102076707149459812e-29 -2.630319821745876056e-28, axis 0 0 1, limit effort=1 velocity=20
- added joint depthcam_servo1: type fixed, parent link_camera_mount, child link_servo_mg, origin xyz=5.5511151231257827021e-17 0 -0.025000000000000022204 rpy=4.3617391034891754833e-16 5.3309457331573694348e-17 -3.141592653589793116, axis 0 0 1, limit effort=1 velocity=20
- added joint depthcam_servo2: type fixed, parent link_camservo_m1, child link_servo_mg_2, origin xyz=2.0431766708101095631e-06 -0.016528097546539638474 -0.034229054784774615161 rpy=-1.57079632679489678 7.3027692487011614622e-18 -1.1102230246251530892e-16, axis 0 0 1, limit effort=1 velocity=20
- added joint depthcam_servo_mount: type fixed, parent link_camera_pole, child link_camera_mount, origin xyz=2.7755575615628913511e-17 0 -0.39999999999999980016 rpy=-1.2617474596870634083e-17 -1.2891945871787910814e-42 1.4001445930311992858e-31, axis 0 0 1, limit effort=1 velocity=20
- added joint display: type fixed, parent link_camera_mount, child link_display, origin xyz=5.5511151231257827021e-17 0.027086138725280789474 -0.012500000000000066613 rpy=1.57079632679489678 1.570796326794896558 0, axis 0 0 1, limit effort=1 velocity=20
- added joint elbow: type revolute, parent link_arm3, child link_arm4, origin xyz=-1.3877787807814456755e-17 -0.13846826553344726562 -0.0090000000000012569945 rpy=4.4665167253899272883e-15 1.553727326119394013e-15 -0.10254325014991327869, axis 0 0 1, limit lower=-2.0943951023931952626 upper=2.0943951023931952626 effort=1 velocity=20
- added joint esp: type fixed, parent link_base, child link_esp, origin xyz=0.034606292843817568206 0.089212568923828047818 0.010000000000000119904 rpy=3.141592653589793116 -4.2598488881936717019e-29 -2.6303198217458904053e-28, axis 0 0 1, limit effort=1 velocity=20
- added joint extension: type fixed, parent link_base, child link_extension, origin xyz=-0.21589470607041608141 0.24645307473837524403 0.010000000000000076536 rpy=-3.141592653589793116 1.5777218104420230503e-29 1.570796326794896558, axis 0 0 1, limit effort=1 velocity=20
- added joint front_left_motor_mount: type fixed, parent link_base, child link_planetary_gear_motor_4, origin xyz=0.201105816066258547 -0.07884444065391765788 -0.010000000000000008882 rpy=1.570796326794896558 -9.4663308626523462545e-30 1.5707963267948972241, axis 0 0 1, limit effort=1 velocity=20
- added joint front_left_wheel: type continuous, parent link_planetary_gear_motor_4, child link_wheel_4, origin xyz=0 0.00013236607255473487044 0.024200000000000027045 rpy=3.141592653589793116 1.5549748421209326805e-16 1.5124586876682719616, axis 0 0 1, limit effort=1 velocity=20
- added joint front_right_motor_mount: type fixed, parent link_base, child link_planetary_gear_motor, origin xyz=-0.27889418393372578109 -0.078844440653917546857 -0.0099999999999997868372 rpy=-1.570796326794896558 -6.3108872417683060394e-30 1.570796326794896558, axis 0 0 1, limit effort=1 velocity=20
- added joint front_right_wheel: type continuous, parent link_planetary_gear_motor, child link_wheel, origin xyz=1.3877787807814456755e-17 0.00013236607255473313571 0.024200000000000054801 rpy=-2.424069566570910828e-15 -1.3601736821082903874e-14 1.4496119042768058627, axis 0 0 1, limit effort=1 velocity=20
- added joint gripper_lastlink: type fixed, parent link_armlast2, child link_gripper_base, origin xyz=2.7755575615628913511e-17 0.014777543023228589814 -0.019999999999999906741 rpy=7.2997163869102196598e-15 1.3877787807814109163e-16 -3.141592653589793116, axis 0 0 1, limit effort=1 velocity=20
- added joint gripper_slider1: type prismatic, parent link_gripper_base, child link_gripper_2, origin xyz=0.0050000190455400661538 -0.0063797864131631132345 -0.010499999999998954614 rpy=1.570796326794896558 7.8825834748385956598e-15 -1.5707963267948956698, axis 0 0 1, limit lower=-0.027000000000000003164 upper=-0.0020000000000000001041 effort=1 velocity=20, mimic joint=gripper_slider2 multiplier=1.0 offset=0.0
- added joint gripper_slider2: type prismatic, parent link_gripper_base, child link_gripper, origin xyz=-0.0049999999671311301519 -0.0063797864131628911899 -0.010499999999998954614 rpy=1.5707963267949074382 -4.0245584642662129694e-15 1.5707963267948952257, axis 0 0 1, limit lower=-0.027000000000000003164 upper=-0.0020000000000000001041 effort=1 velocity=20
- added joint inner_bearing_top_mount: type fixed, parent link_arm1_bearing, child link_arm1_top_mount, origin xyz=-1.0269562977782697999e-15 2.8622937353617317058e-17 -0.0074999999999999719669 rpy=1.9828452313990001816e-18 1.302483993487112669e-18 2.7755575615628538802e-16, axis 0 0 1, limit effort=1 velocity=20
- added joint jetson: type fixed, parent link_base, child link_jetson, origin xyz=0.10316286437116763131 0.21110693215579343085 0.010000000000000008882 rpy=3.141592653589793116 -3.9443045261052524062e-29 -2.6303198217458756076e-28, axis 0 0 1, limit effort=1 velocity=20
- added joint lastlink_aux: type fixed, parent link_armlast, child link_armlast2, origin xyz=-5.5511151231257827021e-17 -0.014777543023228534302 -0.010000000000000064393 rpy=7.7715611723761204349e-16 -1.3739009929736324021e-15 0, axis 0 0 1, limit effort=1 velocity=20
- added joint lidar: type fixed, parent link_base, child link_lidar, origin xyz=-0.038894183933733589287 -0.16928471393882676965 -6.8151522794832716411e-22 rpy=-1.2617474596943606799e-17 -4.2598488881935332536e-29 -2.6303198217458818854e-28, axis 0 0 1, limit effort=1 velocity=20
- added joint link3_motor: type fixed, parent link_wrist_mid, child link_planetary_gear_motor_5, origin xyz=-1.3877787807814456755e-17 0.019050000000000011369 0.01600000000000002115 rpy=-1.5707963267948972241 1.570796326794896336 0, axis 0 0 1, limit effort=1 velocity=20
- added joint motor_wrist2_coupler: type fixed, parent link_motor_horn, child link_wrist_base, origin xyz=1.3877787807814456755e-17 1.9081958235744878039e-17 -0.0039999999999998925304 rpy=-1.3600232051658128177e-15 -1.075528555105610168e-16 -1.57079632679489678, axis 0 0 1, limit effort=1 velocity=20
- added joint pmotor2_fixed: type fixed, parent link_arm3, child link_planetary_gear_motor_7, origin xyz=-1.3877787807814456755e-17 -0.13846826553344726562 -1.3877787807814456755e-17 rpy=-3.141592653589793116 -1.7367564398556450549e-16 1.570796326794896558, axis 0 0 1, limit effort=1 velocity=20
- added joint power_connector: type fixed, parent link_base, child link_power_line_mount, origin xyz=-0.038894183933733672554 0.26162940494715314355 0.010000000000000008882 rpy=-3.141592653589793116 -2.2088105346188310933e-29 3.141592653589793116, axis 0 0 1, limit effort=1 velocity=20
- added joint pwd: type fixed, parent link_base, child link_pdb, origin xyz=-0.093481909483668107486 0.14373710822760596417 0.0099999999999999013289 rpy=-3.141592653589793116 -7.8886090522105048125e-29 1.570796326794896558, axis 0 0 1, limit effort=1 velocity=20
- added joint servo: type fixed, parent link_arm3, child link_planetary_gear_motor_6, origin xyz=4.1633363423443370266e-17 -0.13846826553344726562 -0.050000000000000044409 rpy=1.5535570332398524153e-16 -1.4217996905493939005e-14 1.570796326794896558, axis 0 0 1, limit effort=1 velocity=20
- added joint servo2_wrist3: type fixed, parent link_arm_wrist2, child link_servo_mg_4, origin xyz=0.03854382224380958899 0 -0.013174576908349958093 rpy=1.6653345369377022701e-16 1.5707963267948912289 0, axis 0 0 1, limit effort=1 velocity=20
- added joint servo_wrist2: type fixed, parent link_wrist_end, child link_servo_mg_3, origin xyz=0.020000000000000048989 2.7755575615628913511e-17 -0.062034498560428752434 rpy=-1.57079632679489678 2.2204460492503120948e-16 1.57079632679489678, axis 0 0 1, limit effort=1 velocity=20
- added joint shoulder: type revolute, parent link_arm2, child link_arm3, origin xyz=-0.033380152669139837029 0.02500000000000080283 -0.066448956727981595138 rpy=1.5707963267948921171 -1.4353143270888701899 -3.1415926535897829019, axis 0 0 1, limit lower=-2.0943951023931952626 upper=1.2217304763960306069 effort=1 velocity=20
- added joint ultrasonic_back_left: type fixed, parent link_base, child link_ultrasonic, origin xyz=0.10110581606626183049 0.29615555934607018518 0.0049999999999996635677 rpy=1.570796326794896558 -4.1020767071493280899e-29 -2.628919677152840782e-28, axis 0 0 1, limit effort=1 velocity=20
- added joint ultrasonic_back_right: type fixed, parent link_base, child link_ultrasonic_2, origin xyz=-0.17889418393372902294 0.29615555934607018518 0.0049999999999996635677 rpy=1.570796326794896558 -4.2598488881934637492e-29 -2.628919677152840782e-28, axis 0 0 1, limit effort=1 velocity=20
- added joint ultrasonic_front_left: type fixed, parent link_base, child link_ultrasonic_3, origin xyz=0.10110581606626177498 -0.20384444065391355005 0.0049999999999999012248 rpy=-1.570796326794896558 -4.1020767071494620541e-29 -2.6289196771528497503e-28, axis 0 0 1, limit effort=1 velocity=20
- added joint ultrasonic_front_right: type fixed, parent link_base, child link_ultrasonic_4, origin xyz=-0.1788941839337290507 -0.20384444065391355005 0.0049999999999999012248 rpy=-1.570796326794896558 -4.1020767071494620541e-29 -2.6289196771528497503e-28, axis 0 0 1, limit effort=1 velocity=20
- added joint worm1_armplate: type fixed, parent link_arm_mount_base, child link_wormgearmotor, origin xyz=4.1633363423443370266e-17 1.3877787807814456755e-17 -0.0099999999999999082678 rpy=-5.6472276733811738881e-16 -1.1799182869416098514e-16 3.141592653589793116, axis 0 0 1, limit effort=1 velocity=20
- added joint wormmotor1_fixed: type fixed, parent link_arm2, child link_wormgearmotor_2, origin xyz=-0.033380152669139892541 -0.035000000000000017208 -0.066448956727981595138 rpy=1.570796326794901443 -0.34906585039886572908 9.2342611865085384893e-17, axis 0 0 1, limit effort=1 velocity=20
- added joint wormotor1_fixed: type fixed, parent link_wormgearmotor, child link_arm1_base, origin xyz=3.442956469176805534e-05 -9.5955306764913816941e-05 -0.0091999999999999755584 rpy=-3.2747661034511961278e-16 8.2220102522426096915e-16 -3.141592653589793116, axis 0 0 1, limit effort=1 velocity=20
- added joint wormotor2_fixed: type fixed, parent link_arm2, child link_wormgearmotor_3, origin xyz=-0.033380152669139920296 0.044999999999999998335 -0.066448956727981595138 rpy=1.5707963267948976682 -0.34906585039886567357 9.2342611865096786399e-17, axis 0 0 1, limit effort=1 velocity=20
- added joint wrist1: type revolute, parent link_planetary_gear_motor_5, child link_motor_horn, origin xyz=1.1492543028346347e-16 9.7144514654701197287e-17 0.041674999999999962075 rpy=-3.1415926535897726879 3.1086244689504245081e-15 -1.6211724080414808835, axis 0 0 1, limit lower=-2.0943951023931952626 upper=2.0943951023931952626 effort=1 velocity=20
- added joint wrist1_link2: type fixed, parent link_wrist_base, child link_wrist_end, origin xyz=6.0715321659188248304e-18 -4.1633363423443370266e-17 -0.0070499999999998896882 rpy=3.1918911957974047287e-15 -1.9081958235745149209e-16 -4.8572257327351288897e-17, axis 0 0 1, limit effort=1 velocity=20
- added joint wrist2: type revolute, parent link_servo_mg_3, child link_arm_wrist2, origin xyz=-1.1102230246251565404e-16 4.4408920985006261617e-16 0.0065499999999974085896 rpy=3.141592653589793116 -3.3480163086352534694e-15 1.0635136700377485486, axis 0 0 1, limit lower=-1.570796326794896558 upper=1.570796326794896558 effort=1 velocity=20
- added joint wrist3: type revolute, parent link_servo_mg_4, child link_armlast, origin xyz=2.8622937353617317058e-17 1.6653345369377348106e-16 0.0040499999999998870237 rpy=-3.1415926535897913396 -2.1024848528839129176e-14 0.39282862773488136376, axis 0 0 1, limit lower=-2.0943951023931952626 upper=2.0943951023931952626 effort=1 velocity=20
- joint arm_wrist_bearing_mount: origin xyz=-1.1102230246251565404e-16 0.023400000000000031886 0.016000000000000041966 rpy=1.570796326794896336 -0.45412831300399308931 -3.1415926535897904515 -> xyz=0 0.023400000000000031886 0.01600000000000002115 rpy=1.5707963267948974462 -0.52290389070105258718 3.1415926535897540361
- joint link3_fix_wrist: origin xyz=-5.5511151231257827021e-17 -0.16999999999999998446 -4.1633363423443370266e-17 rpy=-3.1415926535897806815 -1.5939872126258999345e-16 2.7755575615628169023e-16 -> xyz=2.7755575615628913511e-17 -0.11999999999999999556 -5.2041704279304212832e-17 rpy=-3.1415926535897789051 7.1840615370227320013e-16 -5.5511151231258061214e-17
